Commit message: Refine MoveIt workspace split

File: src/zivid_artist_bot/urdf/artist_bot.xacro (robot description, xacro)
@@ -1,5 +1,5 @@
 <?xml version="1.0"?>
-<robot name="iiwa7" xmlns:xacro="http://www.ros.org/wiki/xacro">
-    <xacro:include filename="$(find lbr_description)/urdf/iiwa7/iiwa7_description.xacro" />
+<robot name="iiwa14" xmlns:xacro="http://www.ros.org/wiki/xacro">
+    <xacro:include filename="$(find lbr_description)/urdf/iiwa14/iiwa14_description.xacro" />
     <xacro:arg name="robot_name" default="lbr" />
     <xacro:arg name="mode" default="mock" />
@@ -14,5 +14,5 @@
         <visual>
             <geometry>
-                <mesh filename="package://zivid_artist_bot/meshes/table.stl" scale="0.001 0.001 0.001" />
+                <mesh filename="package://zivid_artist_bot/meshes/table.dae" scale="1 1 1" />
             </geometry>
             <material name="gray">
@@ -22,5 +22,5 @@
         <collision>
             <geometry>
-                <mesh filename="package://zivid_artist_bot/meshes/table.stl" scale="0.001 0.001 0.001" />
+                <mesh filename="package://zivid_artist_bot/meshes/table.dae" scale="1 1 1" />
             </geometry>
         </collision>
@@ -31,15 +31,15 @@
         <origin xyz="0 0 0" rpy="1.5708 0 0" />
     </joint>
-    <xacro:iiwa7
+    <xacro:iiwa14
         robot_name="$(arg robot_name)"
         mode="$(arg mode)"
         system_config_path="$(arg system_config_path)"
         initial_joint_positions_path="$(arg initial_joint_positions_path)" />
-    <joint name="table_to_robot_joint" type="prismatic">
+    <joint name="table_to_robot_joint" type="fixed">
         <parent link="table_link" />
         <child link="$(arg robot_name)_link_0" />
         <axis xyz="0 0 1" />
         <limit lower="-2.0" upper="2.0" effort="10.0" velocity="1.0" />
-        <origin xyz="0 0.04 0" rpy="-1.57079 0 0" />
+        <origin xyz="0 0 0" rpy="-1.5708 1.5708 0" />
     </joint>
 </robot>
