Commit message: changed limits and moveit yaml to reference joint_limit_* convention

File: src/iiwa14_description/urdf/iiwa14/iiwa14.xacro (robot description, xacro)
@@ -1,22 +1,4 @@
 <?xml version="1.0"?>
 <robot xmlns:xacro="http://www.ros.org/wiki/xacro">
-    <xacro:include filename="$(find iiwa14_description)/urdf/iiwa14/iiwa14_description.xacro" />
-    <xacro:arg name="robot_name" default="lbr" />
-    <xacro:arg name="mode" default="mock" />
-    <xacro:arg
-        name="system_config_path"
-        default="$(find iiwa14_description)/ros2_control/lbr_system_config.yaml" />
-    <xacro:arg
-        name="initial_joint_positions_path"
-        default="$(find iiwa14_description)/ros2_control/initial_joint_positions.yaml" />
-    <link name="world" />
-    <joint name="$(arg robot_name)_world_joint" type="fixed">
-        <parent link="world" />
-        <child link="$(arg robot_name)_link_0" />
-    </joint>
-    <xacro:iiwa14
-        robot_name="$(arg robot_name)"
-        mode="$(arg mode)"
-        system_config_path="$(arg system_config_path)"
-        initial_joint_positions_path="$(arg initial_joint_positions_path)" />
+  <xacro:include filename="$(find lbr_description)/urdf/iiwa14/iiwa14.xacro"/>
 </robot>

File: src/iiwa14_description/urdf/iiwa14/iiwa14_description.xacro (robot description, xacro)
@@ -1,4 +1,18 @@
 <?xml version="1.0"?>
-<robot xmlns:xacro="http://www.ros.org/wiki/xacro">
-    <xacro:include filename="/home/mark/ros2_ws/src/lbr_fri_ros2_stack/lbr_description/urdf/iiwa14/iiwa14_description.xacro" />
+<robot name="iiwa14" xmlns:xacro="http://www.ros.org/wiki/xacro">
+  <xacro:include filename="$(find iiwa14_description)/urdf/iiwa14/iiwa14.xacro"/>
+  <xacro:arg name="robot_name" default="lbr"/>
+  <xacro:arg name="mode" default="mock"/>
+  <xacro:arg name="system_config_path" default="$(find iiwa14_description)/ros2_control/lbr_system_config.yaml"/>
+  <xacro:arg name="initial_joint_positions_path" default="$(find iiwa14_description)/ros2_control/initial_joint_positions.yaml"/>
+  <link name="world"/>
+  <joint name="$(arg robot_name)_world_joint" type="fixed">
+    <parent link="world"/>
+    <child link="$(arg robot_name)_link_0"/>
+  </joint>
+  <xacro:iiwa14
+    robot_name="$(arg robot_name)"
+    mode="$(arg mode)"
+    system_config_path="$(arg system_config_path)"
+    initial_joint_positions_path="$(arg initial_joint_positions_path)"/>
 </robot>

File: src/zivid_artist_bot/urdf/artist_bot.xacro (robot description, xacro)
@@ -1,45 +1,45 @@
 <?xml version="1.0"?>
 <robot name="iiwa14" xmlns:xacro="http://www.ros.org/wiki/xacro">
-    <xacro:include filename="$(find lbr_description)/urdf/iiwa14/iiwa14_description.xacro" />
-    <xacro:arg name="robot_name" default="lbr" />
-    <xacro:arg name="mode" default="mock" />
-    <xacro:arg
-        name="system_config_path"
-        default="$(find lbr_description)/ros2_control/lbr_system_config.yaml" />
-    <xacro:arg
-        name="initial_joint_positions_path"
-        default="$(find lbr_description)/ros2_control/initial_joint_positions.yaml" />
-    <link name="world" />
-    <link name="table_link">
-        <visual>
-            <geometry>
-                <mesh filename="package://zivid_artist_bot/meshes/table.dae" scale="1 1 1" />
-            </geometry>
-            <material name="gray">
-                <color rgba="0.8 0.8 0.8 1" />
-            </material>
-        </visual>
-        <collision>
-            <geometry>
-                <mesh filename="package://zivid_artist_bot/meshes/table.dae" scale="1 1 1" />
-            </geometry>
-        </collision>
-    </link>
-    <joint name="world_to_table_joint" type="fixed">
-        <parent link="world" />
-        <child link="table_link" />
-        <origin xyz="0 0 0" rpy="1.5708 0 0" />
-    </joint>
-    <xacro:iiwa14
-        robot_name="$(arg robot_name)"
-        mode="$(arg mode)"
-        system_config_path="$(arg system_config_path)"
-        initial_joint_positions_path="$(arg initial_joint_positions_path)" />
-    <joint name="table_to_robot_joint" type="fixed">
-        <parent link="table_link" />
-        <child link="$(arg robot_name)_link_0" />
-        <axis xyz="0 0 1" />
-        <limit lower="-2.0" upper="2.0" effort="10.0" velocity="1.0" />
-        <origin xyz="0 0 0" rpy="-1.5708 1.5708 0" />
-    </joint>
+  <xacro:include filename="$(find lbr_description)/urdf/iiwa14/iiwa14_description.xacro"/>
+  <xacro:arg name="robot_name" default="lbr"/>
+  <xacro:arg name="mode" default="mock"/>
+  <xacro:arg
+      name="system_config_path"
+      default="$(find lbr_description)/ros2_control/lbr_system_config.yaml"/>
+  <xacro:arg
+      name="initial_joint_positions_path"
+      default="$(find lbr_description)/ros2_control/initial_joint_positions.yaml"/>
+  <link name="world"/>
+  <link name="table_link">
+    <visual>
+      <geometry>
+        <mesh filename="package://zivid_artist_bot/meshes/table.dae" scale="1 1 1"/>
+      </geometry>
+      <material name="gray">
+        <color rgba="0.8 0.8 0.8 1"/>
+      </material>
+    </visual>
+    <collision>
+      <geometry>
+        <mesh filename="package://zivid_artist_bot/meshes/table.dae" scale="1 1 1"/>
+      </geometry>
+    </collision>
+  </link>
+  <joint name="world_to_table_joint" type="fixed">
+    <parent link="world"/>
+    <child link="table_link"/>
+    <origin xyz="0 0 0" rpy="1.5708 0 0"/>
+  </joint>
+  <xacro:iiwa14
+      robot_name="$(arg robot_name)"
+      mode="$(arg mode)"
+      system_config_path="$(arg system_config_path)"
+      initial_joint_positions_path="$(arg initial_joint_positions_path)"/>
+  <joint name="table_to_robot_joint" type="fixed">
+    <parent link="table_link"/>
+    <child link="$(arg robot_name)_link_0"/>
+    <axis xyz="0 0 1" />
+    <limit lower="-2.0" upper="2.0" effort="10.0" velocity="1.0" />
+    <origin xyz="0 0 0" rpy="-1.5708 1.5708 0"/>
+  </joint>
 </robot>
